File: sch/pc88kbd.kicad_pcb (KiCad board)
At the start: 2 copper layers, 29.2 x 17.8 mm, 11 parts, among them X1 CONN-6S, X2 CONN-3

Commit message: element values
Routing:
- net GND: track 61.9 -> 68.2 mm
Changed lines of the file:
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@@
 (kicad_pcb (version 4) (host pcbnew 4.0.7)
   (general
-    (links 25)
+    (links 31)
     (no_connects 0)
     (area 134.390001 50.64 188.060001 89.000001)
     (thickness 1.6)
     (drawings 11)
-    (tracks 56)
+    (tracks 60)
     (zones 0)
     (modules 11)
@@
   )
   (setup
-    (last_trace_width 0.4)
+    (last_trace_width 2)
     (user_trace_width 1)
     (user_trace_width 1.5)
@@
     (mod_text_size 1 1)
     (mod_text_width 0.15)
-    (pad_size 2 2)
-    (pad_drill 0.8)
+    (pad_size 1.9 1.9)
+    (pad_drill 0.9)
     (pad_to_mask_clearance 0.2)
     (aux_axis_origin 0 0)
@@
     (add_net "Net-(R3-Pad1)")
     (add_net VCC)
+  )
+  (module MyLib:Mini_din6 (layer F.Cu)
+    (at 175.26 71.12 90)
+    (tags "MINI DIN")
+    (fp_text reference X1 (at 0 -7.62 90) (layer F.SilkS)
+      (effects (font (thickness 0.3048)))
+    )
+    (fp_text value CONN-6S (at 0 8.89 90) (layer F.SilkS)
+      (effects (font (thickness 0.3048)))
+    )
+    (fp_line (start -6.85 -5.77) (end 6.85 -5.77) (layer F.SilkS) (width 0.381))
+    (fp_line (start 6.85 -5.77) (end 6.85 7.23) (layer F.SilkS) (width 0.381))
+    (fp_line (start 6.85 7.23) (end -6.85 7.23) (layer F.SilkS) (width 0.381))
+    (fp_line (start -6.85 7.23) (end -6.85 -5.77) (layer F.SilkS) (width 0.381))
+    (pad 2 thru_hole circle (at -1.3 -1.25 90) (size 1.9 1.9) (drill 0.9) (layers *.Cu *.Mask F.SilkS))
+    (pad 1 thru_hole circle (at 1.3 -1.25 90) (size 1.9 1.9) (drill 0.9) (layers *.Cu *.Mask F.SilkS)
+      (net 6 "Net-(DD1-Pad5)"))
+    (pad 5 thru_hole circle (at 3.4 -3.75 90) (size 1.9 1.9) (drill 0.9) (layers *.Cu *.Mask F.SilkS)
+      (net 7 "Net-(DD1-Pad6)"))
+    (pad 6 thru_hole circle (at -3.4 -3.75 90) (size 1.9 1.9) (drill 0.9) (layers *.Cu *.Mask F.SilkS))
+    (pad 4 thru_hole circle (at -3.4 -1.25 90) (size 1.9 1.9) (drill 0.9) (layers *.Cu *.Mask F.SilkS)
+      (net 1 VCC))
+    (pad 3 thru_hole circle (at 3.4 -1.25 90) (size 1.9 1.9) (drill 0.9) (layers *.Cu *.Mask F.SilkS)
+      (net 2 GND))
+    (pad S thru_hole rect (at -6.858 0.762 90) (size 2.2 2.2) (drill 0.70104) (layers *.Cu *.SilkS *.Mask)
+      (net 2 GND))
+    (pad S thru_hole rect (at -6.858 2.794 90) (size 2.2 2.2) (drill 0.70104) (layers *.Cu *.SilkS *.Mask)
+      (net 2 GND))
+    (pad S thru_hole rect (at -6.858 1.778 90) (size 2.2 2.2) (drill 0.70104) (layers *.Cu *.SilkS *.Mask)
+      (net 2 GND))
+    (pad S thru_hole rect (at 6.858 0.762 90) (size 2.2 2.2) (drill 0.70104) (layers *.Cu *.SilkS *.Mask)
+      (net 2 GND))
+    (pad S thru_hole rect (at 6.858 2.794 90) (size 2.2 2.2) (drill 0.70104) (layers *.Cu *.SilkS *.Mask)
+      (net 2 GND))
+    (pad S thru_hole rect (at 6.858 1.778 90) (size 2.2 2.2) (drill 0.70104) (layers *.Cu *.SilkS *.Mask)
+      (net 2 GND))
+    (pad S thru_hole rect (at -1.27 2.54 90) (size 2.2 2.2) (drill 0.70104) (layers *.Cu *.SilkS *.Mask)
+      (net 2 GND))
+    (pad S thru_hole rect (at 1.27 2.54 90) (size 2.2 2.2) (drill 0.70104) (layers *.Cu *.SilkS *.Mask)
+      (net 2 GND))
+    (pad S thru_hole rect (at 0 2.54 90) (size 2.2 2.2) (drill 0.70104) (layers *.Cu *.SilkS *.Mask)
+      (net 2 GND))
+    (model /home/las/Dropbox/Work/Kicad/3dpackages/minidin_6.wrl
+      (at (xyz 0 0 0))
+      (scale (xyz 1 1 1))
+      (rotate (xyz 0 0 0))
+    )
   )
   (module Capacitors_ThroughHole:C_Disc_D5.0mm_W2.5mm_P2.50mm (layer F.Cu)
@@
     )
   )
-  (module MyLib:Mini_din6 (layer F.Cu)
-    (at 175.26 71.12 90)
-    (tags "MINI DIN")
-    (fp_text reference X1 (at 0 -7.62 90) (layer F.SilkS)
-      (effects (font (thickness 0.3048)))
-    )
-    (fp_text value CONN-6S (at 0 8.89 90) (layer F.SilkS)
-      (effects (font (thickness 0.3048)))
-    )
-    (fp_line (start -6.85 -5.77) (end 6.85 -5.77) (layer F.SilkS) (width 0.381))
-    (fp_line (start 6.85 -5.77) (end 6.85 7.23) (layer F.SilkS) (width 0.381))
-    (fp_line (start 6.85 7.23) (end -6.85 7.23) (layer F.SilkS) (width 0.381))
-    (fp_line (start -6.85 7.23) (end -6.85 -5.77) (layer F.SilkS) (width 0.381))
-    (pad 2 thru_hole circle (at -1.3 -1.25 90) (size 1.9 1.9) (drill 0.9) (layers *.Cu *.Mask F.SilkS))
-    (pad 1 thru_hole circle (at 1.3 -1.25 90) (size 1.9 1.9) (drill 0.9) (layers *.Cu *.Mask F.SilkS)
-      (net 6 "Net-(DD1-Pad5)"))
-    (pad 5 thru_hole circle (at 3.4 -3.75 90) (size 1.9 1.9) (drill 0.9) (layers *.Cu *.Mask F.SilkS)
-      (net 7 "Net-(DD1-Pad6)"))
-    (pad 6 thru_hole circle (at -3.4 -3.75 90) (size 1.9 1.9) (drill 0.9) (layers *.Cu *.Mask F.SilkS))
-    (pad 4 thru_hole circle (at -3.4 -1.25 90) (size 1.9 1.9) (drill 0.9) (layers *.Cu *.Mask F.SilkS)
-      (net 1 VCC))
-    (pad 3 thru_hole circle (at 3.4 -1.25 90) (size 1.9 1.9) (drill 0.9) (layers *.Cu *.Mask F.SilkS)
-      (net 2 GND))
-    (pad S thru_hole rect (at 0 2.53 90) (size 3.2004 1.99898) (drill 0.508) (layers *.Cu *.SilkS *.Mask)
-      (net 2 GND))
-    (pad S thru_hole rect (at 6.85 1.73 90) (size 2.16916 3.2004) (drill 0.508) (layers *.Cu *.SilkS *.Mask)
-      (net 2 GND))
-    (pad S thru_hole rect (at -6.85 1.73 90) (size 2.16916 3.2004) (drill 0.70104) (layers *.Cu *.SilkS *.Mask)
-      (net 2 GND))
-    (model /home/las/Dropbox/Work/Kicad/3dpackages/minidin_6.wrl
-      (at (xyz 0 0 0))
-      (scale (xyz 1 1 1))
-      (rotate (xyz 0 0 0))
-    )
-  )
   (module Pin_Headers:Pin_Header_Straight_1x03_Pitch2.54mm (layer F.Cu)
     (at 153.67 64.77)
@@
   (segment (start 163.91 67.31) (end 163.91 64.77) (width 1.5) (layer B.Cu) (net 1))
   (segment (start 163.91 64.77) (end 166.37 64.77) (width 1.5) (layer B.Cu) (net 1))
+  (segment (start 176.022 64.262) (end 178.054 64.262) (width 2) (layer B.Cu) (net 2) (status C00000))
+  (segment (start 176.022 77.978) (end 178.054 77.978) (width 2) (layer B.Cu) (net 2) (status C00000))
+  (segment (start 177.8 72.39) (end 177.8 71.12) (width 2) (layer B.Cu) (net 2) (status C00000))
+  (segment (start 174.01 67.72) (end 178.054 67.72) (width 1.5) (layer B.Cu) (net 2) (status 400000))
+  (segment (start 177.8 67.31) (end 178.054 67.31) (width 1.5) (layer B.Cu) (net 2))
+  (segment (start 177.8 67.466) (end 177.8 67.31) (width 1.5) (layer B.Cu) (net 2))
+  (segment (start 178.054 67.72) (end 177.8 67.466) (width 1.5) (layer B.Cu) (net 2))
+  (segment (start 178.054 64.262) (end 178.054 67.31) (width 2) (layer B.Cu) (net 2) (status 400000))
+  (segment (start 178.054 67.31) (end 178.054 69.596) (width 2) (layer B.Cu) (net 2) (status 800000))
+  (segment (start 178.054 69.596) (end 177.8 69.85) (width 2) (layer B.Cu) (net 2) (status C00000))
+  (segment (start 166.37 78.7) (end 177.76 78.7) (width 2) (layer B.Cu) (net 2) (status C00000))
+  (segment (start 177.76 78.7) (end 178.054 78.406) (width 2) (layer B.Cu) (net 2) (status C00000))
+  (segment (start 178.054 78.406) (end 178.054 72.644) (width 2) (layer B.Cu) (net 2) (status C00000))
+  (segment (start 178.054 72.644) (end 177.8 72.39) (width 2) (layer B.Cu) (net 2) (status C00000))
+  (segment (start 177.8 72.39) (end 177.8 69.85) (width 2) (layer B.Cu) (net 2) (status C00000))
   (segment (start 158.75 76.2) (end 158.75 72.39) (width 1.5) (layer B.Cu) (net 2))
   (segment (start 158.75 76.2) (end 158.75 78.7) (width 1.5) (layer B.Cu) (net 2))
@@
   (segment (start 153.67 78.74) (end 153.71 78.7) (width 2) (layer B.Cu) (net 2))
   (segment (start 153.67 69.85) (end 153.67 74.93) (width 2) (layer B.Cu) (net 2))
-  (segment (start 176.22 78.74) (end 166.37 78.74) (width 2) (layer B.Cu) (net 2))
   (segment (start 166.37 78.74) (end 163.83 78.74) (width 2) (layer B.Cu) (net 2))
   (segment (start 163.83 78.74) (end 162.56 78.74) (width 2) (layer B.Cu) (net 2))
-  (segment (start 176.22 78.74) (end 176.99 77.97) (width 2) (layer B.Cu) (net 2))
-  (segment (start 174.01 67.72) (end 177.79 67.72) (width 1.5) (layer B.Cu) (net 2) (status 10))
-  (segment (start 177.8 68.58) (end 177.79 68.58) (width 1.5) (layer B.Cu) (net 2))
-  (segment (start 177.8 67.73) (end 177.8 68.58) (width 1.5) (layer B.Cu) (net 2))
-  (segment (start 177.79 67.72) (end 177.8 67.73) (width 1.5) (layer B.Cu) (net 2))
-  (segment (start 177.79 71.12) (end 177.79 68.58) (width 2) (layer B.Cu) (net 2) (status 10))
-  (segment (start 177.79 68.58) (end 177.79 65.07) (width 2) (layer B.Cu) (net 2) (status 20))
-  (segment (start 177.79 65.07) (end 176.99 64.27) (width 2) (layer B.Cu) (net 2) (status 30))
-  (segment (start 177.79 71.12) (end 177.79 77.17) (width 2) (layer B.Cu) (net 2) (status 30))
-  (segment (start 177.79 77.17) (end 176.99 77.97) (width 2) (layer B.Cu) (net 2) (status 30))
   (segment (start 153.75 69.77) (end 153.67 69.85) (width 1) (layer B.Cu) (net 2))
   (segment (start 161.21 64.77) (end 158.75 64.77) (width 1) (layer B.Cu) (net 3))
