File: sch/pc88kbd.sch (KiCad schematic (older format))
At the start: 11 parts, among them X1 CONN-6S, X2 CONN-3

Commit message: element values
Parts:
- C1: value CAPP -> 10uF
- C2: value CAP -> 0.1uF
- R1, R2, R4, R5: value RES -> 4.7K
- R3: value RES -> 2K
Other:
- note added: "Clock"
- note added: "Data"
- moved on the sheet: R3, R4, R5, VD1
Changed lines of the file:
@@
-$EndComp
-$Comp
-L VCC #PWR01
-U 1 1 5A841941
-P 7000 3100
-F 0 "#PWR01" H 7000 3100 30  0001 C CNN
-F 1 "VCC" H 7000 3175 30  0000 C CNN
-F 2 "" H 7000 3100 60  0000 C CNN
-F 3 "" H 7000 3100 60  0000 C CNN
-	1    7000 3100
-	1    0    0    -1
 $EndComp
 $Comp
@@
 P 4700 2900
 F 0 "R2" H 4700 3000 50  0000 C CNN
-F 1 "RES" H 4700 2800 50  0000 C CNN
+F 1 "4.7K" H 4700 2800 50  0000 C CNN
 F 2 "Resistors_SMD:R_0805_HandSoldering" H 4700 2850 60  0001 C CNN
 F 3 "" H 4700 2850 60  0000 C CNN
@@
 P 4400 2900
 F 0 "R1" H 4400 3000 50  0000 C CNN
-F 1 "RES" H 4400 2800 50  0000 C CNN
+F 1 "4.7K" H 4400 2800 50  0000 C CNN
 F 2 "Resistors_SMD:R_0805_HandSoldering" H 4400 2850 60  0001 C CNN
 F 3 "" H 4400 2850 60  0000 C CNN
@@
 $EndComp
 $Comp
-L VCC #PWR03
-U 1 1 5A841A7C
-P 4700 2600
-F 0 "#PWR03" H 4700 2600 30  0001 C CNN
-F 1 "VCC" H 4700 2675 30  0000 C CNN
-F 2 "" H 4700 2600 60  0000 C CNN
-F 3 "" H 4700 2600 60  0000 C CNN
-	1    4700 2600
-	1    0    0    -1
-$EndComp
-$Comp
-L VCC #PWR04
-U 1 1 5A841A9D
-P 4400 2600
-F 0 "#PWR04" H 4400 2600 30  0001 C CNN
-F 1 "VCC" H 4400 2675 30  0000 C CNN
-F 2 "" H 4400 2600 60  0000 C CNN
-F 3 "" H 4400 2600 60  0000 C CNN
-	1    4400 2600
-	1    0    0    -1
-$EndComp
-$Comp
 L LED VD1
 U 1 1 5A841AD9
-P 5400 4100
-F 0 "VD1" H 5400 4300 50  0000 C CNN
-F 1 "LED" H 5400 4000 50  0000 C CNN
-F 2 "LEDs:LED_D3.0mm" H 5400 4050 60  0001 C CNN
-F 3 "" H 5400 4050 60  0000 C CNN
-	1    5400 4100
+P 5200 4100
+F 0 "VD1" H 5200 4300 50  0000 C CNN
+F 1 "LED" H 5200 4000 50  0000 C CNN
+F 2 "LEDs:LED_D3.0mm" H 5200 4050 60  0001 C CNN
+F 3 "" H 5200 4050 60  0000 C CNN
+	1    5200 4100
 	-1   0    0    -1
 $EndComp
@@
 L RES R3
 U 1 1 5A841BA6
-P 5800 4100
-F 0 "R3" H 5800 4200 50  0000 C CNN
-F 1 "RES" H 5800 4000 50  0000 C CNN
-F 2 "Resistors_SMD:R_0805_HandSoldering" H 5800 4050 60  0001 C CNN
-F 3 "" H 5800 4050 60  0000 C CNN
-	1    5800 4100
-	1    0    0    -1
-$EndComp
-$Comp
-L VCC #PWR05
-U 1 1 5A841D20
-P 4100 2600
-F 0 "#PWR05" H 4100 2600 30  0001 C CNN
-F 1 "VCC" H 4100 2675 30  0000 C CNN
-F 2 "" H 4100 2600 60  0000 C CNN
-F 3 "" H 4100 2600 60  0000 C CNN
-	1    4100 2600
+P 5600 4100
+F 0 "R3" H 5600 4200 50  0000 C CNN
+F 1 "2K" H 5600 4000 50  0000 C CNN
+F 2 "Resistors_SMD:R_0805_HandSoldering" H 5600 4050 60  0001 C CNN
+F 3 "" H 5600 4050 60  0000 C CNN
+	1    5600 4100
 	1    0    0    -1
 $EndComp
@@
 	4700 3100 4700 3500
 Wire Wire Line
-	4200 3500 4800 3500
-Wire Wire Line
-	3900 3600 4800 3600
+	4200 3500 4700 3500
+Wire Wire Line
+	4700 3500 4800 3500
+Wire Wire Line
+	3900 3600 4400 3600
+Wire Wire Line
+	4400 3600 4800 3600
 Wire Wire Line
 	4400 3600 4400 3100
@@
 	4100 3400 3900 3400
 Wire Wire Line
-	4000 3200 4000 4200
+	4000 3200 4000 4000
+Wire Wire Line
+	4000 4000 4000 4200
 Wire Wire Line
 	4000 3200 3900 3200
@@
 L RES R4
 U 1 1 5A842070
-P 6500 2900
-F 0 "R4" H 6500 3000 50  0000 C CNN
-F 1 "RES" H 6500 2800 50  0000 C CNN
-F 2 "Resistors_SMD:R_0805_HandSoldering" H 6500 2850 60  0001 C CNN
-F 3 "" H 6500 2850 60  0000 C CNN
-	1    6500 2900
-	0    -1   -1   0
-$EndComp
-Wire Wire Line
-	6100 3700 6500 3700
-Wire Wire Line
-	6500 3700 6500 3100
-$Comp
-L VCC #PWR07
-U 1 1 5A8420D7
-P 6500 2600
-F 0 "#PWR07" H 6500 2600 30  0001 C CNN
-F 1 "VCC" H 6500 2675 30  0000 C CNN
-F 2 "" H 6500 2600 60  0000 C CNN
-F 3 "" H 6500 2600 60  0000 C CNN
-	1    6500 2600
-	1    0    0    -1
-$EndComp
-Wire Wire Line
-	6500 2600 6500 2700
+P 6400 2900
+F 0 "R4" H 6400 3000 50  0000 C CNN
+F 1 "4.7K" H 6400 2800 50  0000 C CNN
+F 2 "Resistors_SMD:R_0805_HandSoldering" H 6400 2850 60  0001 C CNN
+F 3 "" H 6400 2850 60  0000 C CNN
+	1    6400 2900
+	0    -1   -1   0
+$EndComp
+Wire Wire Line
+	6100 3700 6400 3700
+Wire Wire Line
+	6400 3700 6400 3100
+Wire Wire Line
+	6400 2600 6400 2700
 $Comp
 L RES R5
 U 1 1 5A84213E
-P 6800 2900
-F 0 "R5" H 6800 3000 50  0000 C CNN
-F 1 "RES" H 6800 2800 50  0000 C CNN
-F 2 "Resistors_SMD:R_0805_HandSoldering" H 6800 2850 60  0001 C CNN
-F 3 "" H 6800 2850 60  0000 C CNN
-	1    6800 2900
-	0    -1   -1   0
-$EndComp
-$Comp
-L VCC #PWR08
-U 1 1 5A842198
-P 6800 2600
-F 0 "#PWR08" H 6800 2600 30  0001 C CNN
-F 1 "VCC" H 6800 2675 30  0000 C CNN
-F 2 "" H 6800 2600 60  0000 C CNN
-F 3 "" H 6800 2600 60  0000 C CNN
-	1    6800 2600
-	1    0    0    -1
-$EndComp
-Wire Wire Line
-	6800 2600 6800 2700
+P 6700 2900
+F 0 "R5" H 6700 3000 50  0000 C CNN
+F 1 "4.7K" H 6700 2800 50  0000 C CNN
+F 2 "Resistors_SMD:R_0805_HandSoldering" H 6700 2850 60  0001 C CNN
+F 3 "" H 6700 2850 60  0000 C CNN
+	1    6700 2900
+	0    -1   -1   0
+$EndComp
+Wire Wire Line
+	6700 2600 6700 2700
 Wire Wire Line
 	4100 2600 4100 3400
-$Comp
-L VCC #PWR09
-U 1 1 5A842367
-P 5200 2600
-F 0 "#PWR09" H 5200 2600 30  0001 C CNN
-F 1 "VCC" H 5200 2675 30  0000 C CNN
-F 2 "" H 5200 2600 60  0000 C CNN
-F 3 "" H 5200 2600 60  0000 C CNN
-	1    5200 2600
-	1    0    0    -1
-$EndComp
 $Comp
 L GND #PWR010
@@
 P 5600 2900
 F 0 "C2" H 5600 3025 50  0000 C CNN
-F 1 "CAP" H 5600 2775 50  0000 C CNN
+F 1 "0.1uF" H 5600 2775 50  0000 C CNN
 F 2 "Capacitors_ThroughHole:C_Disc_D5.0mm_W2.5mm_P2.50mm" H 5600 2850 60  0001 C CNN
 F 3 "" H 5600 2850 60  0000 C CNN
@@
 P 5200 2900
 F 0 "C1" H 5200 3025 50  0000 C CNN
-F 1 "CAPP" H 5200 2775 50  0000 C CNN
+F 1 "10uF" H 5200 2775 50  0000 C CNN
 F 2 "Capacitors_ThroughHole:CP_Radial_D5.0mm_P2.50mm" H 5200 2850 60  0001 C CNN
 F 3 "" H 5200 2850 60  0000 C CNN
@@
 $EndComp
 Wire Wire Line
-	5200 3000 5200 3200
+	5200 3000 5200 3100
+Wire Wire Line
+	5200 3100 5200 3200
 Wire Wire Line
 	5600 3000 5600 3100
@@
 Connection ~ 5200 3100
 Wire Wire Line
-	5200 2600 5200 2800
+	5200 2600 5200 2700
+Wire Wire Line
+	5200 2700 5200 2800
 Wire Wire Line
 	5600 2800 5600 2700
@@
 L GND #PWR011
 U 1 1 5A84400D
-P 5200 4200
-F 0 "#PWR011" H 5200 4200 30  0001 C CNN
-F 1 "GND" H 5200 4130 30  0001 C CNN
-F 2 "" H 5200 4200 60  0000 C CNN
-F 3 "" H 5200 4200 60  0000 C CNN
-	1    5200 4200
-	1    0    0    -1
-$EndComp
-Wire Wire Line
-	5200 4200 5200 4100
-Wire Wire Line
-	5200 4100 5300 4100
-Wire Wire Line
-	6000 4100 6200 4100
-Wire Wire Line
-	6100 3500 7100 3500
-Wire Wire Line
-	6800 3100 6800 3500
-Connection ~ 6800 3500
+P 5000 4200
+F 0 "#PWR011" H 5000 4200 30  0001 C CNN
+F 1 "GND" H 5000 4130 30  0001 C CNN
+F 2 "" H 5000 4200 60  0000 C CNN
+F 3 "" H 5000 4200 60  0000 C CNN
+	1    5000 4200
+	1    0    0    -1
+$EndComp
+Wire Wire Line
+	5000 4200 5000 4100
+Wire Wire Line
+	5000 4100 5100 4100
+Wire Wire Line
+	5800 4100 6200 4100
+Wire Wire Line
+	6100 3500 6700 3500
+Wire Wire Line
+	6700 3500 7100 3500
+Wire Wire Line
+	6700 3100 6700 3500
+Connection ~ 6700 3500
 Wire Wire Line
 	6200 4100 6200 3600
@@
 	6200 3600 6100 3600
 Wire Wire Line
-	5500 4100 5600 4100
+	5300 4100 5400 4100
+$Comp
+L VCC #PWR?
+U 1 1 5A880C9B
+P 4100 2600
+F 0 "#PWR?" H 4100 2600 30  0001 C CNN
+F 1 "VCC" H 4100 2700 40  0000 C CNN
+F 2 "" H 4100 2600 60  0000 C CNN
+F 3 "" H 4100 2600 60  0000 C CNN
+	1    4100 2600
+	1    0    0    -1
+$EndComp
+$Comp
+L VCC #PWR?
+U 1 1 5A880CCE
+P 4400 2600
+F 0 "#PWR?" H 4400 2600 30  0001 C CNN
+F 1 "VCC" H 4400 2700 40  0000 C CNN
+F 2 "" H 4400 2600 60  0000 C CNN
+F 3 "" H 4400 2600 60  0000 C CNN
+	1    4400 2600
+	1    0    0    -1
+$EndComp
+$Comp
+L VCC #PWR?
+U 1 1 5A880CFA
+P 4700 2600
+F 0 "#PWR?" H 4700 2600 30  0001 C CNN
+F 1 "VCC" H 4700 2700 40  0000 C CNN
+F 2 "" H 4700 2600 60  0000 C CNN
+F 3 "" H 4700 2600 60  0000 C CNN
+	1    4700 2600
+	1    0    0    -1
+$EndComp
+$Comp
+L VCC #PWR?
+U 1 1 5A880D26
+P 5200 2600
+F 0 "#PWR?" H 5200 2600 30  0001 C CNN
+F 1 "VCC" H 5200 2700 40  0000 C CNN
+F 2 "" H 5200 2600 60  0000 C CNN
+F 3 "" H 5200 2600 60  0000 C CNN
+	1    5200 2600
+	1    0    0    -1
+$EndComp
+$Comp
+L VCC #PWR?
+U 1 1 5A880D68
+P 6400 2600
+F 0 "#PWR?" H 6400 2600 30  0001 C CNN
+F 1 "VCC" H 6400 2700 40  0000 C CNN
+F 2 "" H 6400 2600 60  0000 C CNN
+F 3 "" H 6400 2600 60  0000 C CNN
+	1    6400 2600
+	1    0    0    -1
+$EndComp
+$Comp
+L VCC #PWR?
+U 1 1 5A880D94
+P 6700 2600
+F 0 "#PWR?" H 6700 2600 30  0001 C CNN
+F 1 "VCC" H 6700 2700 40  0000 C CNN
+F 2 "" H 6700 2600 60  0000 C CNN
+F 3 "" H 6700 2600 60  0000 C CNN
+	1    6700 2600
+	1    0    0    -1
+$EndComp
+$Comp
+L VCC #PWR?
+U 1 1 5A880DC0
+P 7000 3100
+F 0 "#PWR?" H 7000 3100 30  0001 C CNN
+F 1 "VCC" H 7000 3200 40  0000 C CNN
+F 2 "" H 7000 3100 60  0000 C CNN
+F 3 "" H 7000 3100 60  0000 C CNN
+	1    7000 3100
+	1    0    0    -1
+$EndComp
+Text Notes 2950 2850 0    60   ~ 0
+Data
+Text Notes 2950 3650 0    60   ~ 0
+Clock
+Text Notes 7550 3550 0    60   ~ 0
+Data
 $EndSCHEMATC
