File: sch/ps2owk.kicad_pcb (KiCad board)
At the start: 2 copper layers, 29.2 x 17.8 mm, 11 parts, among them X1 CONN-6S, X2 CONN-3

Commit message: hw: update schematic
Parts:
- C1: value CAPP -> 10uF
- C2: value CAP -> 0.1uF; footprint Capacitors_ThroughHole:C_Disc_D5.0mm_W2.5mm_P2.50mm -> Capacitors_SMD:C_0805_HandSoldering; moved to B.Cu
- R1, R2, R4, R5: value RES -> 4.7K
- R3: value RES -> 2K
- X1: value CONN-6S -> CONN-6
- X2: value CONN-3 -> CONN-4; footprint Pin_Headers:Pin_Header_Straight_1x03_Pitch2.54mm -> Socket_Strips:Socket_Strip_Straight_1x04_Pitch2.54mm
- moved C2 1.27 mm to (160.0, 76.2)
- moved VD1 1.27 mm to (153.7, 76.2)
Connections:
- X1 pad S: GND -> (no net)
Routing:
- net GND: track 68.2 -> 61.9 mm
- net Net-(R3-Pad1): track 2.46 -> 3.73 mm
