File: sch/ps2owk.sch (KiCad schematic (older format))
At the start: 11 parts, among them X1 CONN-6S, X2 CONN-3

Commit message: hw: update schematic
Parts:
- removed X1: CONN-6S, MyLib:Mini_din6, symbol CONN-6S
- removed X2: CONN-3, Pin_Headers:Pin_Header_Straight_1x03_Pitch2.54mm, symbol CONN-3
- added X1: CONN-6, MyLib:Mini_din6, symbol mylib:CONN-6
- added X2: CONN-4, Socket_Strips:Socket_Strip_Straight_1x04_Pitch2.54mm, symbol mylib:CONN-4
- C1: symbol CAPP -> mylib:CAPP
- C2: footprint Capacitors_ThroughHole:C_Disc_D5.0mm_W2.5mm_P2.50mm -> Capacitors_SMD:C_0805_HandSoldering; symbol CAP -> mylib:CAP
- DD1: symbol ATtiny13 -> mylib:ATtiny13
- R1, R2, R3, R4, R5: symbol RES -> mylib:RES
- VD1: symbol LED -> mylib:LED
Connections:
- net GND: now also X1.3, X2.3, X2.4
- net VCC: now also X1.4, X2.1
- net at DD1.2 (PB3), R5.1: now also X2.2
- net at DD1.5 (PB0), R2.1: now also X1.1
- net at DD1.6 (PB1), R1.1: now also X1.5
Other:
- note added: "+5V"
- note added: "GND"
- moved on the sheet: R3, R4, R5, VD1
